File: unit.kicad_sch (KiCad schematic)
At the start: 81 parts, among them J3 Micro_SD_Card_Det1, J4 Conn_01x03_Socket, J5 SWD, Q1 AO3400A, U1 RT9013, U2 W25Q128JVS, U3 TPS61040DBV, U5 MPU-6050, U6 STM32F407VETx, Y1 8MHz

Commit message: update v1.0
Connections:
- net GND: now also J1.14, J2.13, J2.15; no longer J1.18, J2.30, J2.32
- net OLED_DC: now also J1.12; no longer J1.19
- net PA10: now also J2.10; no longer J2.2
- net PA11: now also J2.11; no longer J1.30
- net PA12: now also J2.12; no longer J1.31
- net PA15: now also J2.32; no longer J1.32
- net PA3: now also J1.30; no longer J1.1
- net PA8: now also J2.8; no longer J1.29
- net PA9: now also J2.9; no longer J2.1
- net PB0: now also J1.27; no longer J1.4
- net PB1: now also J1.26; no longer J1.5
- net PB3: now also J2.25; no longer J2.9
- net PB4: now also J2.24; no longer J2.10
- net PB5: now also J2.23; no longer J2.11
- net PB6: now also J2.22; no longer J2.12
- net PB7: now also J2.21; no longer J2.13
- net PB8: now also J2.20; no longer J2.14
- net PB9: now also J2.19; no longer J2.15
- net PC0: now also J1.6; no longer J2.26
- net PC1: now also J1.7; no longer J2.27
- net PC13: now also J1.3; no longer J2.23
- net PC14: now also J1.4; no longer J2.24
- net PC15: now also J1.5; no longer J2.25
- net PC2: now also J1.8; no longer J2.28
- net PC3: now also J1.9; no longer J2.29
- net PC4: now also J1.29; no longer J1.2
- net PC5: now also J1.28; no longer J1.3
- net PC6: now also J2.6; no longer J1.27
- net PC7: now also J2.7; no longer J1.28
- net PD0: now also J2.31; no longer J2.3
- net PD1: now also J2.30; no longer J2.4
- net PD10: now also J1.10; no longer J1.21
- net PD11: now also J2.1; no longer J1.22
- net PD12: now also J2.2; no longer J1.23
- net PD13: now also J2.3; no longer J1.24
- net PD14: now also J2.4; no longer J1.25
- net PD15: now also J2.5; no longer J1.26
- net PD4: now also J2.29; no longer J2.5
- net PD5: now also J2.28; no longer J2.6
- net PD6: now also J2.27; no longer J2.7
- net PD7: now also J2.26; no longer J2.8
- net PD9: now also J1.11; no longer J1.20
- net PE0: now also J2.18; no longer J2.17
- net PE1: now also J2.17; no longer J2.18
- net PE10: now also J1.22; no longer J1.9
- net PE11: now also J1.21; no longer J1.10
- net PE12: now also J1.20; no longer J1.11
- net PE13: now also J1.19; no longer J1.12
- net PE14: now also J1.18; no longer J1.13
- net PE15: now also J1.17; no longer J1.14
- net PE2: now also J1.31; no longer J2.19
- net PE3: now also J1.32; no longer J2.20
- net PE4: now also J1.1; no longer J2.21
- net PE5: now also J1.2; no longer J2.22
- net PE7: now also J1.25; no longer J1.6
- net PE8: now also J1.24; no longer J1.7
- net PE9: now also J1.23; no longer J1.8
- net VCC: now also J1.13, J2.14; no longer J1.17, J2.31
